Commit message: Robot setting in progress 05.03

File: hair_D/omo_r1/omo_r1_description/urdf/omo_r1.urdf.g2.xacro (robot description, xacro)
@@ -30,11 +30,11 @@
     </inertial>
   </link>
-  <joint name="wheel_left_joint" type="continuous">
+  <!-- <joint name="wheel_left_joint" type="continuous">
     <parent link="base_link"/>
     <child link="wheel_left_link"/>
     <origin xyz="0.0 0.275 0.037" rpy="0.0 0.0 0"/>
     <axis xyz="0 1 0"/>
-  </joint>
-  <link name="wheel_left_link">
+  </joint> -->
+  <!-- <link name="wheel_left_link">
     <visual>
       <origin xyz="-0.1105 -0.06 0.1104" rpy="-1.57 0 0"/>
@@ -57,6 +57,6 @@
                izz="2.0712558e-03" />
       </inertial>
-  </link>
-  <joint name="wheel_right_joint" type="continuous">
+  </link> -->
+  <!-- <joint name="wheel_right_joint" type="continuous">
     <parent link="base_link"/>
     <child link="wheel_right_link"/>
@@ -85,6 +85,6 @@
                izz="2.0712558e-03" />
       </inertial>
-  </link>
-  <joint name="caster_back_right_joint" type="fixed">
+  </link> -->
+  <!-- <joint name="caster_back_right_joint" type="fixed">
     <parent link="base_link"/>
     <child link="caster_back_right_link"/>
@@ -125,11 +125,11 @@
                izz="0.000001" />
     </inertial>
-  </link>
-  <joint name="imu_joint" type="fixed">
+  </link> -->
+  <!-- <joint name="imu_joint" type="fixed">
     <parent link="base_link"/>
     <child link="imu_link"/>
     <origin xyz="0.0 0 0.190" rpy="0 0 1.5758"/>
   </joint>
-  <link name="imu_link"/>
+  <link name="imu_link"/> -->
   <joint name="scan_joint" type="fixed">
     <parent link="base_link"/>
@@ -159,5 +159,5 @@
     </inertial>
   </link>
-  <joint name="camera_joint" type="fixed">
+  <!-- <joint name="camera_joint" type="fixed">
     <origin xyz="0.07 0.0 0.63" rpy="0 0.7 0"/>
     <parent link="base_link"/>
@@ -190,4 +190,4 @@
     <child link="camera_rgb_optical_frame"/>
   </joint>
-  <link name="camera_rgb_optical_frame"/>
+  <link name="camera_rgb_optical_frame"/> -->
 </robot>

Commit message: 05.13

File: hair_D/omo_r1/omo_r1_description/urdf/omo_r1.urdf.g2.xacro (robot description, xacro)
@@ -135,5 +135,5 @@
     <parent link="base_link"/>
     <child link="base_scan"/>
-    <origin xyz="0.06 0 0.230" rpy="0.0 0.0 0.0"/>
+    <origin xyz="0.06 0 0.230" rpy="0.0 0.0 1.0472"/>
   </joint>
   <link name="base_scan">

Commit message: setting 05.25

File: hair_D/omo_r1/omo_r1_description/urdf/omo_r1.urdf.g2.xacro (robot description, xacro)
@@ -135,5 +135,5 @@
     <parent link="base_link"/>
     <child link="base_scan"/>
-    <origin xyz="0.06 0 0.230" rpy="0.0 0.0 1.0472"/>
+    <origin xyz="0.06856 0 0.230" rpy="0.0 0.0 0.0"/>
   </joint>
   <link name="base_scan">

Commit message: 05.26

File: hair_D/omo_r1/omo_r1_description/urdf/omo_r1.urdf.g2.xacro (robot description, xacro)
@@ -135,5 +135,5 @@
     <parent link="base_link"/>
     <child link="base_scan"/>
-    <origin xyz="0.06856 0 0.230" rpy="0.0 0.0 0.0"/>
+    <origin xyz="0.06817 0 0.230" rpy="0.0 0.0 0.0"/>
   </joint>
   <link name="base_scan">

Commit message: 05.29

File: hair_D/omo_r1/omo_r1_description/urdf/omo_r1.urdf.g2.xacro (robot description, xacro)
@@ -126,10 +126,10 @@
     </inertial>
   </link> -->
-  <!-- <joint name="imu_joint" type="fixed">
+  <joint name="imu_joint" type="fixed">
     <parent link="base_link"/>
     <child link="imu_link"/>
-    <origin xyz="0.0 0 0.190" rpy="0 0 1.5758"/>
+    <origin xyz="0.183 0 0.190" rpy="0 0 0"/>
   </joint>
-  <link name="imu_link"/> -->
+  <link name="imu_link"/>
   <joint name="scan_joint" type="fixed">
     <parent link="base_link"/>
